File: keyboard_v1.1/keyboard_v1.0.kicad_pcb (KiCad board)
At the start: 2 copper layers, 100 x 100 mm, 135 parts, among them M3 MountingHole_3.2mm_M3, P1 USB_C_Plug, Q1 AO3400A, Q2 AO3400A, Q3 AO3400A, Q4 AO3400A, SW1 Cherry_MX_1u, SW10 Cherry_MX_1u, SW11 Cherry_MX_1u, SW12 Cherry_MX_1u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

Commit message: 2022-04-12 keyboard v1.1 with generated gerber files
Parts:
- removed D34: 1N5819, Diode_THT:D_DO-41_SOD81_P10.16mm_Horizontal
- D1, R2, R3: moved to B.Cu
- moved C48 290.1 mm to (66.6, 64.2), turned to 180 degrees
- moved C50 278.2 mm to (61.9, 61.2), turned to 90 degrees
- moved R34 269.8 mm to (66.7, 62.2), turned to 180 degrees
- moved D43 267.2 mm to (65.0, 59.4)
- moved C49 260.4 mm to (96.2, 60.8), turned to 180 degrees
- moved D18 251.9 mm to (60.0, 120.0), turned to 180 degrees
- moved D17 250.0 mm to (60.0, 100.0)
- moved D20 246.9 mm to (80.0, 100.0)
- moved L5 244.1 mm to (89.4, 58.9), turned to 180 degrees
- moved R33 244.0 mm to (104.5, 55.2), turned to 180 degrees
- moved R3 241.0 mm to (42.2, 109.9)
- moved C2 237.1 mm to (66.0, 123.5)
- moved L4 234.8 mm to (106.9, 42.9)
- moved C5 234.6 mm to (86.5, 123.5)
- moved D3 230.7 mm to (46.9, 112.6)
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Routing:
- net GND: track 42.3 -> 642.0 mm, vias 2 -> 18
- net 5V_OUT: track 0.00 -> 337.8 mm, vias 0 -> 8
- net Net-(R1-Pad2): track 0.00 -> 90.0 mm, vias 0 -> 1
- net Net-(R3-Pad2): track 0.00 -> 79.4 mm, vias 0 -> 1
- net Net-(C48-Pad1): track 0.00 -> 71.9 mm, vias 0 -> 2
- net SYSTEM_LOAD: track 0.00 -> 68.3 mm, vias 0 -> 2
- net 3rd_Row: track 0.00 -> 68.3 mm, vias 0 -> 1
- net 4th_Column: track 0.00 -> 66.8 mm, vias 0 -> 2
- net Net-(C49-Pad1): track 0.00 -> 58.8 mm
- net 1st_Column: track 0.00 -> 57.8 mm, vias 0 -> 2
- net Net-(C44-Pad2): track 0.00 -> 53.9 mm
- net Net-(C32-Pad1): track 0.00 -> 53.4 mm, vias 0 -> 3
- net 2nd_Row: track 0.00 -> 51.5 mm, vias 0 -> 1
- net 3rd_Column: track 0.00 -> 50.5 mm, vias 0 -> 2
- net Net-(C34-Pad1): track 0.00 -> 39.5 mm, vias 0 -> 2
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- added copper zone on B.Cu, net GND
- added copper zone on F.Cu, net GND
Other:
- board text added: "Custom Mini Keyboard - Török Sámuel"

Commit message: 2022-04-14 added vias and led positions
Parts:
- moved D16 1.80 mm to (60.0, 81.8)
- moved D17 1.80 mm to (60.0, 101.8)
- moved D18 1.80 mm to (60.0, 121.8)
- moved D19 1.80 mm to (80.0, 81.8)
- moved D20 1.80 mm to (80.0, 101.8)
- moved D21 1.80 mm to (80.0, 121.8)
- moved D22 1.80 mm to (100.0, 81.8)
- moved D23 1.80 mm to (100.0, 101.8)
- moved D24 1.80 mm to (100.0, 121.8)
- moved D26 1.80 mm to (120.0, 81.8)
- moved D27 1.80 mm to (120.0, 101.8)
- moved D28 1.80 mm to (120.0, 121.8)
- moved D41 0.21 mm to (100.8, 63.4)
Routing:
- net unconnected-(P1-PadS1): track 0.00 -> 20.6 mm
- net Net-(P1-PadB5): track 0.00 -> 14.3 mm
- net Net-(F1-Pad1): track 41.0 -> 26.8 mm
- net 5V_OUT: track 337.8 -> 340.6 mm
- net LEDS: track 37.0 -> 38.8 mm
- net Net-(D26-Pad2): track 29.2 -> 30.9 mm
- net Net-(D17-Pad2): track 23.5 -> 24.6 mm
- net Net-(D21-Pad2): track 16.4 -> 17.2 mm
- net Net-(D18-Pad2): track 16.4 -> 17.2 mm
- net GND: track 642.0 -> 641.5 mm, vias 18 -> 309

Commit message: 2022.04.21. 22:45
Parts:
- added SW14: SW_DIP_x01, Connector_PinHeader_2.54mm:PinHeader_1x02_P2.54mm_Vertical, F.Cu at (48.1, 82.0)
- added SW15: SW_DIP_x01, Connector_PinHeader_2.54mm:PinHeader_1x02_P2.54mm_Vertical, F.Cu at (48.2, 78.4)
- added SW16: SW_DIP_x01, Connector_PinHeader_2.54mm:PinHeader_1x02_P2.54mm_Vertical, F.Cu at (62.1, 44.3)
- added SW17: SW_DIP_x01, Connector_PinHeader_2.54mm:PinHeader_1x02_P2.54mm_Vertical, F.Cu at (65.8, 44.3)
- C1, C10, C11, C12, C14, C2, C3, C4, C5, C6, C7, C8, D10, D11, D12, D2, D3, D4, D5, D6, D7, D8, D9, R1: moved to B.Cu
- SW13: value 25336NA -> MTS-102
- moved R1 22.1 mm to (59.7, 64.3)
- moved D2 2.46 mm to (47.0, 94.9)
- moved C7 2.19 mm to (105.9, 85.6)
- moved D3 1.64 mm to (47.0, 114.3)
- moved C4 1.23 mm to (86.1, 84.7), turned to -90 degrees
- moved C10 1.23 mm to (106.2, 104.7), turned to 90 degrees
- moved C6 0.98 mm to (86.3, 104.5), turned to 90 degrees
Connections:
- ESP32 pad 15: unconnected-(ESP32-Pad15) -> Net-(ESP32-Pad15)
- ESP32 pad 16: unconnected-(ESP32-Pad16) -> Net-(ESP32-Pad16)
- ESP32 pad 26: unconnected-(ESP32-Pad26) -> Net-(ESP32-Pad26)
- ESP32 pad 27: 1st_Row -> Net-(ESP32-Pad27)
- ESP32 pad 8: unconnected-(ESP32-Pad8) -> 1st_Row
- P1 pad S1: unconnected-(P1-PadS1) -> GND
Routing:
- net GND: track 641.5 -> 710.0 mm, vias 309 -> 306
- net Net-(R2-Pad2): track 16.9 -> 77.1 mm, vias 0 -> 2
- net 2nd_Column: track 36.6 -> 78.8 mm, vias 2 -> 3
- net 3rd_Column: track 50.5 -> 91.2 mm, vias 2 -> 1
- net 4th_Column: track 66.8 -> 107.3 mm, vias 2 -> 3
- net 3.3V_OUT: track 35.3 -> 73.8 mm
- net Net-(ESP32-Pad15): track 0.00 -> 33.8 mm, vias 0 -> 5
- net Net-(ESP32-Pad16): track 0.00 -> 30.1 mm, vias 0 -> 3
- net 5V_OUT: track 340.6 -> 367.6 mm, vias 8 -> 17
- net Net-(R1-Pad2): track 90.0 -> 67.1 mm, vias 1 -> 0
- net unconnected-(P1-PadS1): track 20.6 -> 0.00 mm
- net Net-(ESP32-Pad27): track 0.00 -> 8.91 mm
- net 1st_Row: track 2.84 -> 10.8 mm, vias 0 -> 1
- net Net-(D4-Pad2): track 0.00 -> 4.59 mm
- net Net-(D8-Pad2): track 0.00 -> 4.46 mm
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