File: keyboard_v1.1/esp32.kicad_sch (KiCad schematic)
At the start: 5 parts

Commit message: 2022.04.21. 22:45
Parts:
- added SW14, SW15, SW16, SW17: SW_DIP_x01, Connector_PinHeader_2.54mm:PinHeader_1x02_P2.54mm_Vertical, symbol Switch:SW_DIP_x01
Connections:
- net +3V3: now also SW14.1, SW15.1, SW16.2, SW17.2
- net 1st_Row: now also ESP32.8 (IO15); no longer ESP32.27 (IO0)
- net at ESP32.15 (IO3): now also SW14.2
- net at ESP32.16 (IO46): now also SW15.2
- net at ESP32.26 (IO45): now also SW16.1
- new net: ESP32.27 (IO0), SW17.1
Changed lines of the file:
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@@
+    (stroke (width 0) (type default) (color 0 0 0 0))
+  )
+  (wire (pts (xy 214.63 106.68) (xy 209.55 106.68))
+    (stroke (width 0) (type default) (color 0 0 0 0))
+  )
+  (wire (pts (xy 105.41 119.38) (xy 110.49 119.38))
     (stroke (width 0) (type default) (color 0 0 0 0))
   )
@@
     (stroke (width 0) (type default) (color 0 0 0 0))
   )
+  (wire (pts (xy 144.78 132.08) (xy 125.73 132.08))
+    (stroke (width 0) (type default) (color 0 0 0 0))
+  )
   (wire (pts (xy 127 68.58) (xy 137.16 68.58))
     (stroke (width 0) (type default) (color 0 0 0 0))
@@
     (stroke (width 0) (type default) (color 0 0 0 0))
   )
-  (wire (pts (xy 175.26 106.68) (xy 193.04 106.68))
+  (wire (pts (xy 105.41 132.08) (xy 110.49 132.08))
+    (stroke (width 0) (type default) (color 0 0 0 0))
+  )
+  (wire (pts (xy 170.18 116.84) (xy 170.18 125.73))
     (stroke (width 0) (type default) (color 0 0 0 0))
   )
@@
     (stroke (width 0) (type default) (color 0 0 0 0))
   )
+  (wire (pts (xy 113.03 91.44) (xy 137.16 91.44))
+    (stroke (width 0) (type default) (color 0 0 0 0))
+  )
   (wire (pts (xy 175.26 76.2) (xy 193.04 76.2))
     (stroke (width 0) (type default) (color 0 0 0 0))
   )
+  (wire (pts (xy 170.18 125.73) (xy 177.8 125.73))
+    (stroke (width 0) (type default) (color 0 0 0 0))
+  )
   (wire (pts (xy 116.84 88.9) (xy 137.16 88.9))
     (stroke (width 0) (type default) (color 0 0 0 0))
@@
     (stroke (width 0) (type default) (color 0 0 0 0))
   )
+  (wire (pts (xy 142.24 119.38) (xy 142.24 116.84))
+    (stroke (width 0) (type default) (color 0 0 0 0))
+  )
   (wire (pts (xy 81.28 86.36) (xy 81.28 82.55))
     (stroke (width 0) (type default) (color 0 0 0 0))
   )
+  (wire (pts (xy 175.26 106.68) (xy 194.31 106.68))
+    (stroke (width 0) (type default) (color 0 0 0 0))
+  )
   (wire (pts (xy 81.28 72.39) (xy 90.17 72.39))
     (stroke (width 0) (type default) (color 0 0 0 0))
@@
     (stroke (width 0) (type default) (color 0 0 0 0))
   )
+  (wire (pts (xy 144.78 116.84) (xy 144.78 132.08))
+    (stroke (width 0) (type default) (color 0 0 0 0))
+  )
   (wire (pts (xy 175.26 78.74) (xy 193.04 78.74))
     (stroke (width 0) (type default) (color 0 0 0 0))
@@
     (stroke (width 0) (type default) (color 0 0 0 0))
   )
+  (wire (pts (xy 125.73 119.38) (xy 142.24 119.38))
+    (stroke (width 0) (type default) (color 0 0 0 0))
+  )
   (wire (pts (xy 116.84 81.28) (xy 137.16 81.28))
+    (stroke (width 0) (type default) (color 0 0 0 0))
+  )
+  (wire (pts (xy 196.85 125.73) (xy 193.04 125.73))
     (stroke (width 0) (type default) (color 0 0 0 0))
   )
@@
     )
   )
-  (global_label "1st_Row" (shape input) (at 193.04 106.68 0) (fields_autoplaced)
-    (effects (font (size 1.27 1.27)) (justify left))
-    (property "Intersheet References" "${INTERSHEET_REFS}" (id 0) (at 203.1336 106.6006 0)
-      (effects (font (size 1.27 1.27)) (justify left) hide)
+  (global_label "1st_Row" (shape input) (at 113.03 91.44 180) (fields_autoplaced)
+    (effects (font (size 1.27 1.27)) (justify right))
+    (property "Intersheet References" "${INTERSHEET_REFS}" (id 0) (at 102.9364 91.5194 0)
+      (effects (font (size 1.27 1.27)) (justify right) hide)
     )
   )
@@
     )
     (pin "1")
+  )
+  (symbol (lib_id "Switch:SW_DIP_x01") (at 118.11 132.08 0) (unit 1)
+    (in_bom yes) (on_board yes) (fields_autoplaced)
+    (property "Reference" "SW15" (id 0) (at 118.11 124.46 0))
+    (property "Value" "SW_DIP_x01" (id 1) (at 118.11 127 0))
+    (property "Footprint" "Connector_PinHeader_2.54mm:PinHeader_1x02_P2.54mm_Vertical" (id 2) (at 118.11 132.08 0)
+      (effects (font (size 1.27 1.27)) hide)
+    )
+    (property "Datasheet" "~" (id 3) (at 118.11 132.08 0)
+      (effects (font (size 1.27 1.27)) hide)
+    )
+    (pin "1")
+    (pin "2")
   )
   (symbol (lib_id "Device:R") (at 93.98 76.2 90) (unit 1)
@@
     )
     (property "Datasheet" "" (id 3) (at 81.28 86.36 0)
+      (effects (font (size 1.27 1.27)) hide)
+    )
+    (pin "1")
+  )
+  (symbol (lib_id "power:+3.3V") (at 105.41 119.38 0) (unit 1)
+    (in_bom yes) (on_board yes) (fields_autoplaced)
+    (property "Reference" "#PWR01" (id 0) (at 105.41 123.19 0)
+      (effects (font (size 1.27 1.27)) hide)
+    )
+    (property "Value" "+3.3V" (id 1) (at 105.41 114.3 0))
+    (property "Footprint" "" (id 2) (at 105.41 119.38 0)
+      (effects (font (size 1.27 1.27)) hide)
+    )
+    (property "Datasheet" "" (id 3) (at 105.41 119.38 0)
       (effects (font (size 1.27 1.27)) hide)
     )
@@
     (pin "2")
   )
+  (symbol (lib_id "Switch:SW_DIP_x01") (at 201.93 106.68 0) (unit 1)
+    (in_bom yes) (on_board yes) (fields_autoplaced)
+    (property "Reference" "SW17" (id 0) (at 201.93 99.06 0))
+    (property "Value" "SW_DIP_x01" (id 1) (at 201.93 101.6 0))
+    (property "Footprint" "Connector_PinHeader_2.54mm:PinHeader_1x02_P2.54mm_Vertical" (id 2) (at 201.93 106.68 0)
+      (effects (font (size 1.27 1.27)) hide)
+    )
+    (property "Datasheet" "~" (id 3) (at 201.93 106.68 0)
+      (effects (font (size 1.27 1.27)) hide)
+    )
+    (pin "1")
+    (pin "2")
+  )
+  (symbol (lib_id "power:+3.3V") (at 196.85 125.73 0) (unit 1)
+    (in_bom yes) (on_board yes) (fields_autoplaced)
+    (property "Reference" "#PWR03" (id 0) (at 196.85 129.54 0)
+      (effects (font (size 1.27 1.27)) hide)
+    )
+    (property "Value" "+3.3V" (id 1) (at 196.85 120.65 0))
+    (property "Footprint" "" (id 2) (at 196.85 125.73 0)
+      (effects (font (size 1.27 1.27)) hide)
+    )
+    (property "Datasheet" "" (id 3) (at 196.85 125.73 0)
+      (effects (font (size 1.27 1.27)) hide)
+    )
+    (pin "1")
+  )
+  (symbol (lib_id "power:+3.3V") (at 105.41 132.08 0) (unit 1)
+    (in_bom yes) (on_board yes) (fields_autoplaced)
+    (property "Reference" "#PWR02" (id 0) (at 105.41 135.89 0)
+      (effects (font (size 1.27 1.27)) hide)
+    )
+    (property "Value" "+3.3V" (id 1) (at 105.41 127 0))
+    (property "Footprint" "" (id 2) (at 105.41 132.08 0)
+      (effects (font (size 1.27 1.27)) hide)
+    )
+    (property "Datasheet" "" (id 3) (at 105.41 132.08 0)
+      (effects (font (size 1.27 1.27)) hide)
+    )
+    (pin "1")
+  )
   (symbol (lib_id "Device:C") (at 71.12 78.74 0) (unit 1)
     (in_bom yes) (on_board yes) (fields_autoplaced)
@@
     (pin "1")
   )
+  (symbol (lib_id "power:+3.3V") (at 214.63 106.68 0) (unit 1)
+    (in_bom yes) (on_board yes) (fields_autoplaced)
+    (property "Reference" "#PWR04" (id 0) (at 214.63 110.49 0)
+      (effects (font (size 1.27 1.27)) hide)
+    )
+    (property "Value" "+3.3V" (id 1) (at 214.63 101.6 0))
+    (property "Footprint" "" (id 2) (at 214.63 106.68 0)
+      (effects (font (size 1.27 1.27)) hide)
+    )
+    (property "Datasheet" "" (id 3) (at 214.63 106.68 0)
+      (effects (font (size 1.27 1.27)) hide)
+    )
+    (pin "1")
+  )
   (symbol (lib_id "Device:C") (at 81.28 78.74 0) (unit 1)
     (in_bom yes) (on_board yes) (fields_autoplaced)
@@
     )
     (property "Datasheet" "~" (id 3) (at 81.28 78.74 0)
+      (effects (font (size 1.27 1.27)) hide)
+    )
+    (pin "1")
+    (pin "2")
+  )
+  (symbol (lib_id "Switch:SW_DIP_x01") (at 118.11 119.38 0) (unit 1)
+    (in_bom yes) (on_board yes) (fields_autoplaced)
+    (property "Reference" "SW14" (id 0) (at 118.11 111.76 0))
+    (property "Value" "SW_DIP_x01" (id 1) (at 118.11 114.3 0))
+    (property "Footprint" "Connector_PinHeader_2.54mm:PinHeader_1x02_P2.54mm_Vertical" (id 2) (at 118.11 119.38 0)
+      (effects (font (size 1.27 1.27)) hide)
+    )
+    (property "Datasheet" "~" (id 3) (at 118.11 119.38 0)
       (effects (font (size 1.27 1.27)) hide)
     )
@@
     (pin "1")
   )
+  (symbol (lib_id "Switch:SW_DIP_x01") (at 185.42 125.73 0) (unit 1)
+    (in_bom yes) (on_board yes) (fields_autoplaced)
+    (property "Reference" "SW16" (id 0) (at 185.42 118.11 0))
+    (property "Value" "SW_DIP_x01" (id 1) (at 185.42 120.65 0))
+    (property "Footprint" "Connector_PinHeader_2.54mm:PinHeader_1x02_P2.54mm_Vertical" (id 2) (at 185.42 125.73 0)
+      (effects (font (size 1.27 1.27)) hide)
+    )
+    (property "Datasheet" "~" (id 3) (at 185.42 125.73 0)
+      (effects (font (size 1.27 1.27)) hide)
+    )
+    (pin "1")
+    (pin "2")
+  )
 )

Commit message: PCB layout done - 2022.07.25.
Parts:
- removed SW14, SW15, SW16, SW17: SW_DIP_x01, Connector_PinHeader_2.54mm:PinHeader_1x02_P2.54mm_Vertical, symbol Switch:SW_DIP_x01
- added JP1, JP2, JP3, JP4: Jumper_3_Bridged12, Connector_PinHeader_2.54mm:PinHeader_1x03_P2.54mm_Horizontal, symbol Jumper:Jumper_3_Bridged12
- added R6, R7, R8, R9: 10K, Resistor_SMD:R_0805_2012Metric_Pad1.20x1.40mm_HandSolder, symbol Device:R
Connections:
- net +3V3: now also JP1.1 (A), JP2.1 (A), JP3.1 (A), JP4.1 (A)
- net 1st_Column: now also ESP32.7 (IO7); no longer ESP32.4 (IO4)
- net 2nd_Column: now also ESP32.6 (IO6); no longer ESP32.5 (IO5)
- net 3rd_Column: now also ESP32.5 (IO5); no longer ESP32.6 (IO6)
- net 4th_Column: now also ESP32.4 (IO4); no longer ESP32.7 (IO7)
- net GND: now also R6.1, R7.1, R8.1, R9.1
- net at ESP32.16 (IO46): now also JP2.2 (C)
- net at ESP32.15 (IO3): now also JP1.2 (C)
- net at ESP32.26 (IO45): now also JP3.2 (C)
- net at ESP32.27 (IO0): now also JP4.2 (C)
- new net: JP3.3 (B), R8.2
- new net: JP4.3 (B), R9.2
- new net: JP2.3 (B), R7.2
- new net: JP1.3 (B), R6.2

Commit message: Corrections on PCB design - 2022.08.04.
Connections:
- net GND: now also JP1.3 (B), JP2.3 (B), JP3.3 (B), JP4.3 (B); no longer R6.1, R7.1, R8.1, R9.1
- net at ESP32.15 (IO3): now also R6.1; no longer JP1.2 (C)
- net at ESP32.16 (IO46): now also R7.2; no longer JP2.2 (C)
- net at ESP32.26 (IO45): now also R8.1; no longer JP3.2 (C)
- net at ESP32.27 (IO0): now also R9.2; no longer JP4.2 (C)
- net at R8.2: now also JP3.2 (C); no longer JP3.3 (B)
- net at R6.2: now also JP1.2 (C); no longer JP1.3 (B)
- new net: JP4.2 (C), R9.1
- new net: JP2.2 (C), R7.1
Other:
- moved on the sheet: R6, R7, R8, R9

Commit message: Firmware added
Parts:
- C20: value 0,1 uF -> 1 uF
Changed lines of the file:
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@@
       (effects (font (size 1.27 1.27)) (justify left))
     )
-    (property "Value" "0,1 uF" (id 1) (at 85.09 80.0099 0)
+    (property "Value" "1 uF" (id 1) (at 85.09 80.0099 0)
       (effects (font (size 1.27 1.27)) (justify left))
     )
