File: keyboard_v1.1/usb-c.kicad_sch (KiCad schematic)
At the start: 4 parts, among them P1 USB_C_Plug

Commit message: 2022.04.21. 22:45
Connections:
- net GND: now also P1.S1 (SHIELD)
Changed lines of the file:
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@@
+    (stroke (width 0) (type default) (color 0 0 0 0))
+  )
+  (wire (pts (xy 104.14 116.84) (xy 104.14 120.65))
     (stroke (width 0) (type default) (color 0 0 0 0))
   )
@@
     )
   )
+  (symbol (lib_id "power:GND") (at 104.14 120.65 0) (unit 1)
+    (in_bom yes) (on_board yes) (fields_autoplaced)
+    (property "Reference" "#PWR0113" (id 0) (at 104.14 127 0)
+      (effects (font (size 1.27 1.27)) hide)
+    )
+    (property "Value" "GND" (id 1) (at 104.14 125.73 0))
+    (property "Footprint" "" (id 2) (at 104.14 120.65 0)
+      (effects (font (size 1.27 1.27)) hide)
+    )
+    (property "Datasheet" "" (id 3) (at 104.14 120.65 0)
+      (effects (font (size 1.27 1.27)) hide)
+    )
+    (pin "1")
+  )
   (symbol (lib_id "Device:R") (at 152.4 59.69 0) (unit 1)
