File: keyboard_v1.1/ws2812b.kicad_sch (KiCad schematic)
At the start: 24 parts

Commit message: PCB layout done - 2022.07.25.
Changed lines of the file:
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@@
   (junction (at 127 19.05) (diameter 0) (color 0 0 0 0)
-  )
-  (junction (at 180.34 78.74) (diameter 0) (color 0 0 0 0)
   )
   (junction (at 88.9 93.98) (diameter 0) (color 0 0 0 0)
   )
   (junction (at 50.8 19.05) (diameter 0) (color 0 0 0 0)
+  )
+  (junction (at 180.34 78.74) (diameter 0) (color 0 0 0 0)
   )
   (junction (at 142.24 78.74) (diameter 0) (color 0 0 0 0)
@@
   )
   (wire (pts (xy 147.32 71.12) (xy 170.18 71.12))
+    (stroke (width 0) (type default) (color 0 0 0 0))
+  )
+  (wire (pts (xy 177.8 78.74) (xy 180.34 78.74))
     (stroke (width 0) (type default) (color 0 0 0 0))
   )
@@
     (stroke (width 0) (type default) (color 0 0 0 0))
   )
-  (wire (pts (xy 180.34 78.74) (xy 177.8 78.74))
-    (stroke (width 0) (type default) (color 0 0 0 0))
-  )
